File: pcb/actual pcb design/rustyjack-h616/sheets/storage_emmc.kicad_sch (KiCad schematic)
At the start: 8 parts, among them J1 Micro_SD_Card, U1 THGBMNG5D1LBAIL

Commit message: everything
Parts:
- J1: footprint Voltlog:microSD_card -> Connector_Card:microSD_HC_Hirose_DM3AT-SF-PEJM5
- U1: footprint Voltlog:WFBGA153 -> projectlib:THGBMNG5D1LBAIL_WFBGA153; symbol emmc-adapter-rescue:THGBMNG5D1LBAIL-voltlog -> H616_lib:THGBMNG5D1LBAIL
- V1: value VOLTLOG_LOGO -> H616_LOGO; footprint Voltlog:voltlog_mask_3mm -> (none); symbol emmc-adapter-rescue:VOLTLOG_LOGO-voltlog -> H616_lib:H616_LOGO; now left out of the parts list
Other:
- title: Voltlog eMMC to microSD Adapter -> H616 eMMC Storage
Changed lines of the file:
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@@
 	(paper "A4")
 	(title_block
-		(title "Voltlog eMMC to microSD Adapter")
+		(title "H616 eMMC Storage")
 		(date "2021-07-06")
 		(rev "A")
@@
 	)
 	(symbol
-		(lib_id "emmc-adapter-rescue:THGBMNG5D1LBAIL-voltlog")
+		(lib_id "H616_lib:THGBMNG5D1LBAIL")
 		(at 137.16 72.39 0)
 		(unit 1)
@@
 			)
 		)
-		(property "Footprint" "Voltlog:WFBGA153"
+		(property "Footprint" "projectlib:THGBMNG5D1LBAIL_WFBGA153"
 			(at 135.89 93.98 0)
 			(effects
@@
 			)
 		)
-		(property "Datasheet" "https://datasheet.lcsc.com/szlcsc/1912111437_KIOXIA-THGBMDG5D1LBAIL_C391254.pdf"
+		(property "Datasheet" "https://lcsc.com/datasheet/lcsc_datasheet_1912111437_TOSHIBA-THGBMNG5D1LBAIL_C391255.pdf"
 			(at 135.89 93.98 0)
 			(effects
@@
 		)
 		(instances
-			(project "emmc-adapter"
+			(project "rustyjack-h616"
 				(path "/68663db6-c703-4253-b388-4008f4be15fd"
 					(reference "U1")
@@
 			)
 		)
-		(property "Footprint" "Voltlog:microSD_card"
+		(property "Footprint" "Connector_Card:microSD_HC_Hirose_DM3AT-SF-PEJM5"
 			(at 237.49 58.42 0)
 			(effects
@@
 		)
 		(instances
-			(project "emmc-adapter"
+			(project "rustyjack-h616"
 				(path "/68663db6-c703-4253-b388-4008f4be15fd"
 					(reference "J1")
@@
 	)
 	(symbol
-		(lib_id "emmc-adapter-rescue:VOLTLOG_LOGO-voltlog")
+		(lib_id "H616_lib:H616_LOGO")
 		(at 182.88 172.72 0)
 		(unit 1)
-		(exclude_from_sim no)
-		(in_bom yes)
-		(on_board yes)
+		(exclude_from_sim yes)
+		(in_bom no)
+		(on_board no)
 		(dnp no)
 		(property "Reference" "V1"
@@
 			)
 		)
-		(property "Value" "VOLTLOG_LOGO"
+		(property "Value" "H616_LOGO"
 			(at 182.88 169.418 0)
 			(effects
@@
 			)
 		)
-		(property "Footprint" "Voltlog:voltlog_mask_3mm"
+		(property "Footprint" ""
 			(at 182.88 172.72 0)
 			(effects
@@
 		)
 		(instances
-			(project "emmc-adapter"
+			(project "rustyjack-h616"
 				(path "/68663db6-c703-4253-b388-4008f4be15fd"
 					(reference "V1")
@@
 		)
 		(instances
-			(project "emmc-adapter"
+			(project "rustyjack-h616"
 				(path "/68663db6-c703-4253-b388-4008f4be15fd"
 					(reference "FID1")
@@
 		)
 		(instances
-			(project "emmc-adapter"
+			(project "rustyjack-h616"
 				(path "/68663db6-c703-4253-b388-4008f4be15fd"
 					(reference "FID2")
@@
 		)
 		(instances
-			(project "emmc-adapter"
+			(project "rustyjack-h616"
 				(path "/68663db6-c703-4253-b388-4008f4be15fd"
 					(reference "FID3")
@@
 		)
 		(instances
-			(project "emmc-adapter"
+			(project "rustyjack-h616"
 				(path "/68663db6-c703-4253-b388-4008f4be15fd"
 					(reference "C2")
@@
 	)
 	(symbol
-		(lib_id "emmc-adapter-rescue:GND-power")
+		(lib_id "H616_emmc-rescue:GND-power")
 		(at 157.48 74.93 0)
 		(unit 1)
@@
 		)
 		(instances
-			(project "emmc-adapter"
+			(project "rustyjack-h616"
 				(path "/68663db6-c703-4253-b388-4008f4be15fd"
 					(reference "#PWR0101")
@@
 	)
 	(symbol
-		(lib_id "emmc-adapter-rescue:VCC-power")
+		(lib_id "H616_emmc-rescue:VCC-power")
 		(at 157.48 67.31 0)
 		(unit 1)
@@
 		)
 		(instances
-			(project "emmc-adapter"
+			(project "rustyjack-h616"
 				(path "/68663db6-c703-4253-b388-4008f4be15fd"
 					(reference "#PWR0102")
@@
 		)
 		(instances
-			(project "emmc-adapter"
+			(project "rustyjack-h616"
 				(path "/68663db6-c703-4253-b388-4008f4be15fd"
 					(reference "C1")
@@
 	)
 	(symbol
-		(lib_id "emmc-adapter-rescue:GND-power")
+		(lib_id "H616_emmc-rescue:GND-power")
 		(at 116.84 102.87 0)
 		(unit 1)
@@
 		)
 		(instances
-			(project "emmc-adapter"
+			(project "rustyjack-h616"
 				(path "/68663db6-c703-4253-b388-4008f4be15fd"
 					(reference "#PWR0103")
