File: pcb/actual pcb design/rustyjack-h616/sheets/wifi_aw859a.kicad_sch (KiCad schematic)
At the start: 1 part

Commit message: everything
Parts:
- U_WIFI1: footprint (none) -> projectlib:AW859A_SMD-44_12X12_P0.9mm
Changed lines of the file:
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@@
 			)
 		)
-		(property "Footprint" ""
+		(property "Footprint" "projectlib:AW859A_SMD-44_12X12_P0.9mm"
 			(at 0 0 0)
 			(effects
@@
 			)
 		)
-		(property "Datasheet" ""
+		(property "Datasheet" "https://linux-sunxi.org/images/1/1f/AW859A_SPEC_V1.4.pdf"
 			(at 0 0 0)
 			(effects
